Commit message: Split into threads and created main app

File: panda_with_sensor.urdf (robot description, URDF)
Before this commit: robot panda, 13 links, 12 joints
Links:
- added link panda_wrist_sensor_link, mass 0.001
Joints:
- added joint wrist_sensor_joint: type fixed, parent panda_link7, child panda_wrist_sensor_link, origin xyz=0 0 0 rpy=0 0 0
- joint panda_hand_joint: parent panda_link8 -> panda_wrist_sensor_link

Commit message: Threading working, control of arm moved to controller.py

File: panda_with_sensor.urdf (robot description, URDF)
Before this commit: robot panda, 14 links, 13 joints
Joints:
- joint wrist_sensor_joint: parent panda_link7 -> panda_link8
